File: koyomi-lvds-hat.kicad_pcb (KiCad board)
At the start: 2 copper layers, 65 x 56.5 mm, 26 parts, among them IC1 SN75LVDS83B, J1 RPi_GPIO, J2 20374-R30E-31, J3 aux_sig, J4 qwiic, J5 Conn_01x06, J6 Conn_01x06, J7 Conn_01x06, U1 AP2114H-2.5

Commit message: RPi/breakout garden standard header with IO22 as INT and IO25 added on top; RGB tracks moved around a bit but length-matched anew
Parts:
- added J8: i2c, Connector_PinSocket_2.54mm:PinSocket_1x06_P2.54mm_Vertical, F.Cu at (147.1, 31.3)
Connections:
- J1 pad 15: unconnected-(J1-BCM22-Pad15) -> GP22
- J1 pad 22: unconnected-(J1-BCM25-Pad22) -> GP25
Routing:
- net GP22: track 0.00 -> 54.5 mm, vias 0 -> 4
- net GP25: track 0.00 -> 38.5 mm, vias 0 -> 1
- net R4: track 53.8 -> 59.2 mm
- net +3V3: track 282.2 -> 286.5 mm
- net SCL: track 77.8 -> 80.2 mm, vias 2 -> 1
- net EN: track 72.0 -> 73.6 mm
- net R5: track 47.8 -> 48.9 mm
- net GND: track 3.57 -> 2.91 mm
- net SDA: track 74.5 -> 74.7 mm, vias 2 -> 1

Commit message: Added silkscreen markings for all the headers
Other:
- board text added: "3V3 PI0 PI1 INS GND"
- board text added: "C1 C2 C3 C4 C5 C6"
- board text added: "GND 3V3 SDA(23) SCL(24) x x"
- board text added: "GND G25 SCL(24) SDA(23) 3V3 G22"
- board text added: "SCL SDA 3V3 GND"
- board text added: "VAD x GND 5V G26 G27"
Changed lines of the file:
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@@
     )
   )
+  (gr_rect (start 150.92 35.97) (end 157.55 42.6)
+    (stroke (width 0.15) (type default)) (fill none) (layer "B.SilkS"))
   (gr_line (start 91 60) (end 91 75.5)
     (stroke (width 0.1) (type solid)) (layer "Edge.Cuts"))
@@
   (gr_line (start 156 25) (end 156 75.5)
     (stroke (width 0.1) (type solid)) (layer "Edge.Cuts"))
+  (gr_text "SCL\nSDA\n3V3\nGND" (at 154.94 42.4) (layer "B.SilkS")
+    (effects (font (size 1 1) (thickness 0.15)) (justify left bottom mirror))
+  )
+  (gr_text "C1\nC2\nC3\nC4\nC5\nC6" (at 139.9 68.33 270) (layer "B.SilkS")
+    (effects (font (size 1.5 1.5) (thickness 0.2)) (justify left bottom mirror))
+  )
+  (gr_text "3V3\nPI0\nPI1\nINS\nGND" (at 112.82 74.84 90) (layer "B.SilkS")
+    (effects (font (size 1.5 1.5) (thickness 0.2)) (justify right bottom mirror))
+  )
+  (gr_text "GND\n3V3\nSDA(23)\nSCL(24)\nx\nx" (at 136.54 65.15) (layer "B.SilkS")
+    (effects (font (size 1.5 1.5) (thickness 0.2)) (justify left bottom mirror))
+  )
   (gr_text "Project Koyomi\nLVDS hat v1\nby Exentio" (at 111.2 47.2) (layer "B.SilkS")
     (effects (font (size 1 1) (thickness 0.2) bold) (justify left bottom mirror))
   )
+  (gr_text "VAD\nx\nGND\n5V\nG26\nG27\n" (at 140.01 48.11 270) (layer "B.SilkS")
+    (effects (font (size 1.5 1.5) (thickness 0.2)) (justify right bottom mirror))
+  )
+  (gr_text "GND\nG25\nSCL(24)\nSDA(23)\n3V3\nG22" (at 145.93 44.59) (layer "B.SilkS")
+    (effects (font (size 1.5 1.5) (thickness 0.2)) (justify left bottom mirror))
+  )
   (gr_text "Project Koyomi\nLVDS hat v1\nby Exentio" (at 99.6 47.1) (layer "F.SilkS")
