File: koyomi-lvds-hat.kicad_pcb (KiCad board)
At the start: 2 copper layers, 65 x 56.5 mm, 35 parts, among them IC1 SN75LVDS83B, J1 RPi_GPIO, J2 20374-R30E-31, J3 aux_sig, J4 qwiic, J5 Conn_01x06, J6 Conn_01x06, J7 Conn_01x06, J8 i2c, U1 AP2114H-2.5

Commit message: v1.2: Murata DLP2ADN121HL4L footprint cleanup, JLCPCB CPL fixes
Other:
- board text added: "Project Koyomi LVDS hat v1.2 by Exentio"
- board text removed: "Project Koyomi LVDS hat v1.1 by Exentio"
